File: preamp_k2/preamp_k2.kicad_pcb (KiCad board)
At the start: 2 copper layers, 40 x 40 mm, 23 parts, among them J1 AudioJack_Stereo, J2 AudioJack_Stereo, J3 9VDC, Q1 BC549, Q2 BC559, Q3 BC549

Commit message: Add files via upload
Parts:
- added C8: 220p, User_Proto_Friendly:C_Disc_T3.0mm_P5.0, F.Cu at (64.3, 60.3)
- C3, C6: value 10u -> 22u
- J4: footprint User_Proto_Friendly:PinHeader_1x02_P2.54mm_Vertical -> User_Global_Library:PinHeader_1x02_P2.54mm_Vertical
- moved Q1 3.82 mm to (57.3, 67.4)
- moved Q2 0.63 mm to (61.4, 57.6)
- moved R1 0.63 mm to (53.8, 57.1)
Connections:
- net Net-(C2-Pad1) renamed /IN
- net Net-(C5-Pad2) renamed /OUT
Routing:
- net Net-(Q2-E): track 53.7 -> 62.8 mm
- net Net-(Q1-C): track 11.7 -> 18.0 mm
- net Net-(Q1-E): track 29.8 -> 33.8 mm
- net Net-(Q2-C): track 13.2 -> 16.1 mm
- net Net-(Q1-B): track 35.1 -> 37.2 mm
Other:
- board text added: "NPN"
- board text added: "PNP"
