File: preamp_k1/preamp_k1.kicad_pcb (KiCad board)
At the start: 2 copper layers, 40 x 40 mm, 18 parts, among them J1 AudioJack_Stereo, J2 AudioJack_Stereo, J3 9VDC, Q1 BC549, Q2 BC549

Commit message: Add files via upload
Parts:
- J4: footprint User_Proto_Friendly:PinHeader_1x02_P2.54mm_Vertical -> User_Global_Library:PinHeader_1x02_P2.54mm_Vertical
Connections:
- net Net-(C1-Pad1) renamed /IN
- net Net-(C2-Pad2) renamed /OUT
