File: preamp_k1/preamp_k1.kicad_sch (KiCad schematic)
At the start: 18 parts, among them J1 AudioJack_Stereo, J2 AudioJack_Stereo, J3 9VDC, Q1 BC549, Q2 BC549

Commit message: Add files via upload
Parts:
- added R8: 0.000001R, User_Proto_Friendly:R_Axial_L6.3mm_D2.5mm_P10.16mm_Horiz, symbol USER_Proto_Friendly:R
- added V1: 8.5V, symbol Simulation_SPICE:VDC
- added V3: VSIN, symbol Simulation_SPICE:VSIN
- J4: footprint User_Proto_Friendly:PinHeader_1x02_P2.54mm_Vertical -> User_Global_Library:PinHeader_1x02_P2.54mm_Vertical
Connections:
- net 0V: now also R8.2, V1.2, V3.2
- net V+: now also V1.1
- net IN: now reaches C1.1, J1.T
- net IN: now also V3.1
- net OUT: now reaches C2.2, J2.T
- new net 0: R8.1
Other:
- note added: "(Not part of the actual circuit)"
- note added: "1. Click on Inspect->Simulator 2. Select an Analysis tab 3. Click the Run triangle"
- note added: "Simulation"
- moved on the sheet: C1, C2, C3, C4, C5, R1, R2, R3, R4, R5, R6, R7
