File: poweramp_k1/poweramp_k1.kicad_pcb (KiCad board)
At the start: 2 copper layers, 40 x 40 mm, 31 parts, among them J1 AudioJack_Stereo, J3 9VDC, J5 SPEAKER, Q1 BC547, Q2 BC337-25, Q3 BC557, Q4 BC327-25, Q5 BC547, Q6 BC547

Commit message: Add files via upload
Parts:
- added C6: 100u, User_Proto_Friendly:CP_Radial_D6.3mm_P2.50mm, F.Cu at (53.8, 57.1)
- C3: footprint User_Proto_Friendly:CP_Radial_D6.3mm_P2.50mm -> User_Proto_Friendly:CP_Radial_D5.0mm_P2.50mm
- D1, D2, D3: footprint User_Proto_Friendly:Diode-DO-35_1.75mmDia_3.4mmWidth_P7.62mm -> User_Proto_Friendly:Diode-DO-35_1.75mmDia_P3.81mm_Vert_CathodeUp
- R1, R11, R12, R13, R2, R3, R4, R5, R6, R7, R8, R9: footprint User_Proto_Friendly:R_Axial_L6.3mm_D2.5mm_P10.16mm_Horiz -> User_Proto_Friendly:R_Axial_L6.3mm_D2.5mm_P3.81mm_Vertical
- moved R8 100.9 mm to (87.8, 56.5), turned to -90 degrees
- moved R12 99.8 mm to (84.6, 60.3), turned to 90 degrees
- moved R7 97.0 mm to (84.0, 53.0)
- moved R13 92.6 mm to (78.6, 69.7), turned to 90 degrees
- moved R5 87.0 mm to (75.7, 58.5), turned to -90 degrees
- moved R9 85.4 mm to (72.2, 61.6), turned to 180 degrees
- moved R6 82.9 mm to (71.7, 66.0)
- moved R3 76.5 mm to (64.7, 66.0)
- moved Q5 76.4 mm to (75.4, 54.6)
- moved R4 76.1 mm to (64.9, 62.7), turned to 90 degrees
- moved R2 75.0 mm to (63.5, 45.4), turned to 180 degrees
- moved C2 73.9 mm to (80.2, 60.6), turned to 90 degrees
- moved R1 71.3 mm to (60.0, 42.2)
- moved J5 70.0 mm to (79.0, 40.0), turned to 180 degrees
- moved R11 67.8 mm to (53.5, 63.9), turned to -90 degrees
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Routing:
- net V+: track 0.00 -> 101.9 mm
- net Net-(Q1-C): track 0.00 -> 33.9 mm
- net Net-(Q1-B): track 0.00 -> 26.2 mm, vias 0 -> 1
- net Net-(C4-Pad2): track 0.00 -> 25.4 mm, vias 0 -> 2
- net /IN: track 0.00 -> 24.2 mm
- net Net-(D1-A): track 0.00 -> 23.1 mm
- net Net-(Q6-B): track 0.00 -> 22.5 mm
- net Net-(D2-K): track 0.00 -> 20.0 mm
- net Net-(C3-Pad1): track 0.00 -> 15.4 mm
- net Net-(Q2-E): track 0.00 -> 14.0 mm
- net /OUT: track 0.00 -> 14.0 mm
- net Net-(C1-Pad1): track 0.00 -> 13.5 mm
- net Net-(Q5-B): track 0.00 -> 13.0 mm
- net Net-(Q1-E): track 0.00 -> 12.0 mm
- net Net-(Q4-E): track 0.00 -> 9.62 mm
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Other:
- board text added: "GND"
- board text added: "VOL"
- board text removed: "NPN"
- board text removed: "OUTPUT"
