File: poweramp_k1/poweramp_k1.kicad_sch (KiCad schematic)
At the start: 35 parts, among them J1 AudioJack_Stereo, J3 9VDC, J5 SPEAKER, Q1 BC547, Q2 BC337-25, Q3 BC557, Q4 BC327-25, Q5 BC547, Q6 BC547

Commit message: Add files via upload
Parts:
- added C6: 100u, User_Proto_Friendly:CP_Radial_D6.3mm_P2.50mm, symbol USER_Proto_Friendly:C_Polarized_Small
- C3: footprint User_Proto_Friendly:CP_Radial_D6.3mm_P2.50mm -> User_Proto_Friendly:CP_Radial_D5.0mm_P2.50mm
- D1, D2, D3: footprint User_Proto_Friendly:Diode-DO-35_1.75mmDia_3.4mmWidth_P7.62mm -> User_Proto_Friendly:Diode-DO-35_1.75mmDia_P3.81mm_Vert_CathodeUp
- R1, R11, R12, R13, R2, R3, R4, R5, R6, R7, R8, R9: footprint User_Proto_Friendly:R_Axial_L6.3mm_D2.5mm_P10.16mm_Horiz -> User_Proto_Friendly:R_Axial_L6.3mm_D2.5mm_P3.81mm_Vertical
Connections:
- net 0V: now also C6.2
- net V+: now also C6.1
Changed lines of the file:
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@@
 	)
 	(junction
+		(at 146.05 20.32)
+		(diameter 0)
+		(color 0 0 0 0)
+	)
+	(junction
 		(at 71.12 44.45)
 		(diameter 0)
@@
 	(wire
 		(pts
+			(xy 153.67 22.86) (xy 153.67 20.32)
+		)
+		(stroke
+			(width 0)
+			(type default)
+		)
+	)
+	(wire
+		(pts
 			(xy 43.18 105.41) (xy 43.18 107.95)
 		)
@@
 	(wire
 		(pts
+			(xy 153.67 20.32) (xy 146.05 20.32)
+		)
+		(stroke
+			(width 0)
+			(type default)
+		)
+	)
+	(wire
+		(pts
 			(xy 104.14 77.47) (xy 104.14 81.28)
 		)
@@
 			)
 		)
-		(property "Footprint" "User_Proto_Friendly:R_Axial_L6.3mm_D2.5mm_P10.16mm_Horiz"
+		(property "Footprint" "User_Proto_Friendly:R_Axial_L6.3mm_D2.5mm_P3.81mm_Vertical"
 			(at 112.776 70.358 90)
 			(hide yes)
@@
 			)
 		)
-		(property "Footprint" "User_Proto_Friendly:R_Axial_L6.3mm_D2.5mm_P10.16mm_Horiz"
+		(property "Footprint" "User_Proto_Friendly:R_Axial_L6.3mm_D2.5mm_P3.81mm_Vertical"
 			(at 97.536 72.898 90)
 			(hide yes)
@@
 			)
 		)
-		(property "Footprint" "User_Proto_Friendly:R_Axial_L6.3mm_D2.5mm_P10.16mm_Horiz"
+		(property "Footprint" "User_Proto_Friendly:R_Axial_L6.3mm_D2.5mm_P3.81mm_Vertical"
 			(at 139.446 48.768 90)
 			(hide yes)
@@
 			)
 		)
-		(property "Footprint" "User_Proto_Friendly:R_Axial_L6.3mm_D2.5mm_P10.16mm_Horiz"
+		(property "Footprint" "User_Proto_Friendly:R_Axial_L6.3mm_D2.5mm_P3.81mm_Vertical"
 			(at 112.268 59.944 90)
 			(hide yes)
@@
 			)
 		)
-		(property "Footprint" "User_Proto_Friendly:R_Axial_L6.3mm_D2.5mm_P10.16mm_Horiz"
+		(property "Footprint" "User_Proto_Friendly:R_Axial_L6.3mm_D2.5mm_P3.81mm_Vertical"
 			(at 64.516 60.198 90)
 			(hide yes)
@@
 			)
 		)
-		(property "Footprint" "User_Proto_Friendly:R_Axial_L6.3mm_D2.5mm_P10.16mm_Horiz"
+		(property "Footprint" "User_Proto_Friendly:R_Axial_L6.3mm_D2.5mm_P3.81mm_Vertical"
 			(at 83.566 60.198 90)
 			(hide yes)
@@
 			)
 		)
-		(property "Footprint" "User_Proto_Friendly:R_Axial_L6.3mm_D2.5mm_P10.16mm_Horiz"
+		(property "Footprint" "User_Proto_Friendly:R_Axial_L6.3mm_D2.5mm_P3.81mm_Vertical"
 			(at 125.984 81.788 90)
 			(hide yes)
@@
 			)
 		)
-		(property "Footprint" "User_Proto_Friendly:CP_Radial_D6.3mm_P2.50mm"
+		(property "Footprint" "User_Proto_Friendly:CP_Radial_D5.0mm_P2.50mm"
 			(at 61.468 50.546 0)
 			(hide yes)
@@
 			)
 		)
-		(property "Footprint" "User_Proto_Friendly:R_Axial_L6.3mm_D2.5mm_P10.16mm_Horiz"
+		(property "Footprint" "User_Proto_Friendly:R_Axial_L6.3mm_D2.5mm_P3.81mm_Vertical"
 			(at 64.516 37.338 90)
 			(hide yes)
@@
 			)
 		)
-		(property "Footprint" "User_Proto_Friendly:R_Axial_L6.3mm_D2.5mm_P10.16mm_Horiz"
+		(property "Footprint" "User_Proto_Friendly:R_Axial_L6.3mm_D2.5mm_P3.81mm_Vertical"
 			(at 64.516 27.178 90)
 			(hide yes)
@@
 			)
 		)
-		(property "Footprint" "User_Proto_Friendly:R_Axial_L6.3mm_D2.5mm_P10.16mm_Horiz"
+		(property "Footprint" "User_Proto_Friendly:R_Axial_L6.3mm_D2.5mm_P3.81mm_Vertical"
 			(at 126.746 90.678 90)
 			(hide yes)
@@
 			)
 		)
-		(property "Footprint" "User_Proto_Friendly:Diode-DO-35_1.75mmDia_3.4mmWidth_P7.62mm"
+		(property "Footprint" "User_Proto_Friendly:Diode-DO-35_1.75mmDia_P3.81mm_Vert_CathodeUp"
 			(at 139.7 63.5 0)
 			(hide yes)
@@
 			)
 		)
-		(property "Footprint" "User_Proto_Friendly:R_Axial_L6.3mm_D2.5mm_P10.16mm_Horiz"
+		(property "Footprint" "User_Proto_Friendly:R_Axial_L6.3mm_D2.5mm_P3.81mm_Vertical"
 			(at 94.234 24.638 90)
 			(hide yes)
@@
 	)
 	(symbol
+		(lib_id "USER_Proto_Friendly:C_Polarized_Small")
+		(at 153.67 25.4 0)
+		(unit 1)
+		(body_style 1)
+		(exclude_from_sim no)
+		(in_bom yes)
+		(on_board yes)
+		(in_pos_files yes)
+		(dnp no)
+		(property "Reference" "C6"
+			(at 156.21 23.5838 0)
+			(show_name no)
+			(do_not_autoplace no)
+			(effects
+				(font
+					(size 1.27 1.27)
+				)
+				(justify left)
+			)
+		)
+		(property "Value" "100u"
+			(at 156.21 26.1238 0)
+			(show_name no)
+			(do_not_autoplace no)
+			(effects
+				(font
+					(size 1.27 1.27)
+				)
+				(justify left)
+			)
+		)
+		(property "Footprint" "User_Proto_Friendly:CP_Radial_D6.3mm_P2.50mm"
+			(at 156.972 39.116 0)
+			(hide yes)
+			(show_name no)
+			(do_not_autoplace no)
+			(effects
+				(font
+					(size 1.27 1.27)
+				)
+			)
+		)
+		(property "Datasheet" ""
+			(at 153.67 25.4 0)
+			(hide yes)
+			(show_name no)
+			(do_not_autoplace no)
+			(effects
+				(font
+					(size 1.27 1.27)
+				)
+			)
+		)
+		(property "Description" "Polarized capacitor, small symbol"
+			(at 156.464 36.068 0)
+			(hide yes)
+			(show_name no)
+			(do_not_autoplace no)
+			(effects
+				(font
+					(size 1.27 1.27)
+				)
+			)
+		)
+		(pin "2"
+		)
+		(pin "1"
+		)
+		(instances
+			(project "poweramp_k1"
+				(path "/17e655d6-68e2-45a0-92e7-3164f3a0bcee"
+					(reference "C6")
+					(unit 1)
+				)
+			)
+		)
+	)
+	(symbol
 		(lib_id "USER_Proto_Friendly:BC557-PNP")
 		(at 130.81 31.75 0)
@@
 	)
 	(symbol
+		(lib_id "User_Global_Symbol_Library:0V")
+		(at 153.67 27.94 0)
+		(unit 1)
+		(body_style 1)
+		(exclude_from_sim no)
+		(in_bom yes)
+		(on_board yes)
+		(in_pos_files yes)
+		(dnp no)
+		(property "Reference" "#PWR025"
+			(at 153.67 33.02 0)
+			(hide yes)
+			(show_name no)
+			(do_not_autoplace no)
+			(effects
+				(font
+					(size 1.27 1.27)
+				)
+			)
+		)
+		(property "Value" "0V"
+			(at 153.67 30.734 0)
+			(show_name no)
+			(do_not_autoplace no)
+			(effects
+				(font
+					(size 1.27 1.27)
+				)
+			)
+		)
+		(property "Footprint" ""
+			(at 153.67 27.94 0)
+			(hide yes)
+			(show_name no)
+			(do_not_autoplace no)
+			(effects
+				(font
+					(size 1.27 1.27)
+				)
+			)
+		)
+		(property "Datasheet" ""
+			(at 153.67 27.94 0)
+			(hide yes)
+			(show_name no)
+			(do_not_autoplace no)
+			(effects
+				(font
+					(size 1.27 1.27)
+				)
+			)
+		)
+		(property "Description" "Power symbol creates a global label with name \"0V\""
+			(at 153.67 27.94 0)
+			(hide yes)
+			(show_name no)
+			(do_not_autoplace no)
+			(effects
+				(font
+					(size 1.27 1.27)
+				)
+			)
+		)
+		(pin "1"
+		)
+		(instances
+			(project "poweramp_k1"
+				(path "/17e655d6-68e2-45a0-92e7-3164f3a0bcee"
+					(reference "#PWR025")
+					(unit 1)
+				)
+			)
+		)
+	)
+	(symbol
 		(lib_id "Simulation_SPICE:VSIN")
 		(at 43.18 113.03 0)
@@
 			)
 		)
-		(property "Footprint" "User_Proto_Friendly:Diode-DO-35_1.75mmDia_3.4mmWidth_P7.62mm"
+		(property "Footprint" "User_Proto_Friendly:Diode-DO-35_1.75mmDia_P3.81mm_Vert_CathodeUp"
 			(at 139.7 46.99 0)
 			(hide yes)
@@
 			)
 		)
-		(property "Footprint" "User_Proto_Friendly:Diode-DO-35_1.75mmDia_3.4mmWidth_P7.62mm"
+		(property "Footprint" "User_Proto_Friendly:Diode-DO-35_1.75mmDia_P3.81mm_Vert_CathodeUp"
 			(at 125.73 91.44 0)
 			(hide yes)
@@
 			)
 		)
-		(property "Footprint" "User_Proto_Friendly:R_Axial_L6.3mm_D2.5mm_P10.16mm_Horiz"
+		(property "Footprint" "User_Proto_Friendly:R_Axial_L6.3mm_D2.5mm_P3.81mm_Vertical"
 			(at 139.446 60.198 90)
 			(hide yes)
